File: IRremote.brd (EAGLE design)
At the start: 31.5 x 75.5 mm, 12 parts

Commit message: 1.1
1.1
Parts:
- moved BAT 1.02 mm to (17.5, 6.65), turned to 180 degrees
Routing:
- net GND: track 119.5 -> 112.9 mm
- net N$5: track 72.4 -> 69.6 mm
- net 11: track 44.6 -> 42.8 mm
- net 12: track 50.1 -> 48.6 mm
- net VCC: track 34.5 -> 34.2 mm, vias 1 -> 0
- net VDD: track 50.8 -> 51.0 mm, vias 0 -> 2
