File: IRremote.sch (EAGLE design)
At the start: 12 parts

Commit message: 1.1
1.1
Other:
- moved on the sheet: BAT-1
Changed lines of the file:
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@@
 <instance part="R4" gate="G$1" x="-48.26" y="96.52" rot="R90"/>
 <instance part="GND5" gate="1" x="78.74" y="71.12" rot="R90"/>
-<instance part="BAT" gate="-1" x="99.06" y="104.14" rot="R90"/>
+<instance part="BAT" gate="-1" x="83.82" y="91.44" rot="R270"/>
 <instance part="BAT" gate="-2" x="93.98" y="109.22" rot="R270"/>
 <instance part="VDD1" gate="G$1" x="81.28" y="76.2" rot="R270"/>
@@
 </segment>
 <segment>
+<pinref part="VDD2" gate="G$1" pin="VDD"/>
 <pinref part="BAT" gate="-2" pin="S"/>
-<pinref part="VDD2" gate="G$1" pin="VDD"/>
 </segment>
 </net>
 <net name="N$5" class="1">
 <segment>
-<pinref part="BAT" gate="-1" pin="S"/>
-<wire x1="99.06" y1="101.6" x2="99.06" y2="91.44" width="0.1524" layer="91"/>
-<wire x1="99.06" y1="91.44" x2="83.82" y2="91.44" width="0.1524" layer="91"/>
-<wire x1="83.82" y1="91.44" x2="83.82" y2="119.38" width="0.1524" layer="91"/>
+<wire x1="83.82" y1="91.44" x2="83.82" y2="93.98" width="0.1524" layer="91"/>
 <pinref part="S2" gate="1" pin="2"/>
+<wire x1="83.82" y1="93.98" x2="83.82" y2="119.38" width="0.1524" layer="91"/>
 <wire x1="83.82" y1="119.38" x2="73.66" y2="119.38" width="0.1524" layer="91"/>
 <wire x1="73.66" y1="119.38" x2="73.66" y2="111.76" width="0.1524" layer="91"/>
-<wire x1="99.06" y1="71.12" x2="99.06" y2="91.44" width="0.1524" layer="91"/>
-<junction x="99.06" y="91.44"/>
+<pinref part="BAT" gate="-1" pin="S"/>
+<junction x="83.82" y="93.98"/>
 </segment>
 </net>
